File: FEU2.brd (EAGLE design)
At the start: 160 x 100 mm, 48 parts, among them IC1 LM358N, Q1 8M, Q2 32748

Commit message: BRD 1
Parts:
- moved R23 180.1 mm to (111.4, 69.9), flipped to the bottom, turned to 270 degrees
- moved R25 176.6 mm to (117.7, 72.1), turned to 90 degrees
- moved U$4 173.0 mm to (103.9, 75.3), flipped to the bottom
- moved C13 169.1 mm to (112.6, 64.4), turned to 180 degrees
- moved R24 152.7 mm to (105.6, 64.7), flipped to the bottom, turned to 90 degrees
- moved D1 149.2 mm to (92.1, 72.8), turned to 270 degrees
- moved C11 136.1 mm to (111.4, 75.8), flipped to the bottom, turned to 90 degrees
- moved C5 130.5 mm to (54.3, 38.3), flipped to the bottom
- moved C12 123.1 mm to (101.3, 64.3), flipped to the bottom, turned to 180 degrees
- moved C4 120.9 mm to (43.5, 36.9), flipped to the bottom, turned to 90 degrees
- moved SB2 117.5 mm to (47.6, 52.7)
- moved C3 112.7 mm to (39.8, 36.3), flipped to the bottom, turned to 180 degrees
- moved R7 105.9 mm to (35.0, 29.1), flipped to the bottom, turned to 270 degrees
- moved C9 103.7 mm to (41.4, 58.7), flipped to the bottom
- moved UART_USB 103.6 mm to (68.9, 47.7), turned to 270 degrees
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
Commit message: BRD 2
Parts:
- moved R10 84.9 mm to (9.74, 79.1), turned to 270 degrees
- moved SWD 83.8 mm to (32.0, 4.51)
- moved UART_USB 54.1 mm to (31.0, 86.2), turned to 0 degrees
- moved C11 45.4 mm to (66.1, 76.8)
- moved D1 45.4 mm to (46.8, 73.8)
- moved R23 45.4 mm to (66.1, 70.9)
- moved R24 45.4 mm to (60.2, 65.8)
- moved R25 45.4 mm to (72.3, 73.1)
- moved U$4 45.4 mm to (58.5, 76.3)
- moved C12 45.4 mm to (56.0, 65.4)
- moved L2 45.4 mm to (36.8, 72.6)
- moved C13 45.4 mm to (67.3, 65.4)
- moved S1 38.5 mm to (56.0, 52.4)
- moved R11 33.0 mm to (57.9, 4.08)
- moved SB2 29.7 mm to (23.0, 36.1)
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Routing:
- net GND: track 0.00 -> 485.7 mm, vias 0 -> 6
- net 3.3V: track 0.00 -> 233.8 mm, vias 0 -> 2
- net USB+: track 0.00 -> 158.8 mm, vias 0 -> 4
- net NRST: track 0.00 -> 158.0 mm, vias 0 -> 2
- net 15V: track 0.00 -> 121.0 mm
- net BLUE: track 0.00 -> 104.6 mm
- net N$23: track 0.00 -> 103.1 mm
- net WHITE: track 0.00 -> 101.7 mm
- net V_LED: track 0.00 -> 74.6 mm, vias 0 -> 2
- net N$4: track 0.00 -> 72.8 mm, vias 0 -> 2
- net N$31: track 0.00 -> 69.3 mm
- net SWCLK: track 0.00 -> 46.9 mm, vias 0 -> 2
- net N$7: track 0.00 -> 45.0 mm
- net N$3: track 0.00 -> 37.8 mm
- net SWDAT: track 0.00 -> 37.0 mm, vias 0 -> 2
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
Commit message: BRD 3
Parts:
- moved FEU1 11.3 mm to (13.8, 16.4)
- moved FEU2 10.8 mm to (14.1, 23.8)
- moved U$3 9.95 mm to (7.06, 7.53)
- moved R7 9.32 mm to (14.8, 8.45)
Connections:
- removed net DAC: U$1.14
- net S3: now also U$1.14; no longer U$1.11
Routing:
- net ADC_RES: track 0.00 -> 142.1 mm, vias 0 -> 2
- net USART_RX_STM: track 10.6 -> 136.1 mm, vias 0 -> 2
- net UART_TX_STM: track 9.96 -> 126.5 mm, vias 0 -> 2
- net 15V: track 121.0 -> 223.2 mm, vias 0 -> 2
- net ADC_S: track 27.2 -> 90.9 mm, vias 0 -> 2
- net S3: track 13.9 -> 73.9 mm, vias 0 -> 2
- net GND: track 485.7 -> 534.3 mm, vias 6 -> 7
- net N$23: track 103.1 -> 115.7 mm
- net BLUE: track 104.6 -> 97.9 mm
- net WHITE: track 101.7 -> 95.6 mm

Commit message: BRD 4
Parts:
- moved R10 76.1 mm to (25.5, 4.59), turned to 0 degrees
- moved SB1 29.5 mm to (22.8, 31.5)
- moved C14 18.4 mm to (8.89, 42.5), turned to 0 degrees
- moved R11 11.4 mm to (69.2, 4.08)
- moved R9 9.73 mm to (8.43, 37.2), turned to 180 degrees
- moved SWD 7.82 mm to (39.8, 4.35)
- moved C7 0.85 mm to (35.0, 33.8), turned to 90 degrees
- moved SB2 0.22 mm to (22.8, 36.1)
Routing:
- net N$5: track 19.2 -> 73.4 mm
- net ADC_RES: track 142.1 -> 90.2 mm
- net 3.3V: track 233.8 -> 197.9 mm
- net GND: track 534.3 -> 499.1 mm, vias 7 -> 2
- net N$17: track 10.8 -> 42.4 mm
- net N$7: track 45.0 -> 24.4 mm
- net ADC_S: track 90.9 -> 105.4 mm, vias 2 -> 4
- net BLUE: track 97.9 -> 109.2 mm
- net WHITE: track 95.6 -> 107.0 mm
- net SWCLK: track 46.9 -> 54.8 mm
- net NRST: track 158.0 -> 150.2 mm
- net S3: track 73.9 -> 67.4 mm
- net 15V: track 223.2 -> 228.2 mm
- net N$3: track 37.8 -> 39.6 mm
- net SWDAT: track 37.0 -> 38.1 mm

Commit message: BRD 5
Parts:
- R15: device resistor:R0805 -> resistor:R1206
- R6: device resistor:M1206 -> resistor:R1206
- R9: device resistor:M1206 -> resistor:R0805
- moved S1 37.7 mm to (18.4, 55.0)
- moved R4 37.1 mm to (58.5, 28.2)
- moved C9 35.8 mm to (25.9, 55.0), turned to 90 degrees
- moved UART_USB 31.6 mm to (62.1, 81.1)
- moved LED1 31.4 mm to (5.43, 51.3), turned to 90 degrees
- moved R6 29.7 mm to (18.1, 34.4), turned to 270 degrees
- moved C11 21.3 mm to (44.8, 76.6)
- moved C12 21.3 mm to (34.7, 65.2)
- moved C13 21.3 mm to (46.0, 65.2)
- moved R23 21.3 mm to (44.8, 70.7)
- moved R25 21.3 mm to (51.0, 72.9)
- moved D1 21.3 mm to (25.5, 73.5)
- moved L2 21.3 mm to (15.5, 72.4)
- moved R24 21.3 mm to (39.0, 65.5)
- moved U$4 21.3 mm to (37.2, 76.1)
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Routing:
- net UART_TX_STM: track 126.5 -> 57.7 mm, vias 2 -> 0
- net USART_RX_STM: track 136.1 -> 70.5 mm, vias 2 -> 0
- net 3.3V: track 197.9 -> 254.2 mm, vias 2 -> 4
- net N$5: track 73.4 -> 129.5 mm
- net V_LED: track 74.6 -> 19.6 mm, vias 2 -> 0
- net ADC_S: track 105.4 -> 153.4 mm
- net GND: track 499.1 -> 539.0 mm, vias 2 -> 4
- net 15V: track 228.2 -> 267.6 mm, vias 2 -> 4
- net NRST: track 150.2 -> 187.9 mm
- net ADC_RES: track 90.2 -> 125.8 mm, vias 2 -> 4
- net USB+: track 158.8 -> 130.6 mm, vias 4 -> 2
- net N$4: track 72.8 -> 96.0 mm
- net SWCLK: track 54.8 -> 34.9 mm
- net N$23: track 115.6 -> 95.9 mm
- net N$3: track 39.6 -> 28.9 mm
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
Commit message: BRD 6
Parts:
- moved UART_USB 6.99 mm to (66.8, 75.9), turned to 270 degrees
- moved L2 1.58 mm to (16.8, 71.4)
- moved R13 0.58 mm to (30.2, 42.5)
- moved C10 0.50 mm to (49.5, 49.3)
Routing:
- net N$31: track 69.3 -> 23.9 mm
- net 15V: track 267.6 -> 232.1 mm
- net USB+: track 130.6 -> 164.9 mm
- net GND: track 539.0 -> 557.1 mm
- net 3.3V: track 254.2 -> 262.8 mm
- net USART_RX_STM: track 70.5 -> 64.8 mm
- net N$23: track 95.9 -> 91.5 mm
- net UART_TX_STM: track 57.7 -> 54.2 mm
- net ADC_S: track 153.4 -> 156.4 mm
- net NRST: track 187.9 -> 190.9 mm
- net WHITE: track 100.2 -> 101.7 mm
- net ADC_RES: track 125.8 -> 126.9 mm
- net BLUE: track 103.2 -> 104.3 mm
- net N$4: track 96.0 -> 95.1 mm
- net S3: track 61.3 -> 61.9 mm
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Other:
- board text added: "+"
- board text added: "3.3V"
- board text added: "5V"
- board text added: "GND"
- board text added: "_"

Commit message: BRD 7
Other:
- board size 160 x 100 mm -> 79.4 x 81.7 mm
- board text added: "RX"
- board text added: "TX"
Changed lines of the file:
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@@
 <board>
 <plain>
-<wire x1="0" y1="0" x2="160" y2="0" width="0" layer="20"/>
-<wire x1="160" y1="0" x2="160" y2="100" width="0" layer="20"/>
-<wire x1="160" y1="100" x2="0" y2="100" width="0" layer="20"/>
-<wire x1="0" y1="100" x2="0" y2="0" width="0" layer="20"/>
-<text x="75.56" y="70.26" size="1.778" layer="16" rot="MR270">_</text>
-<text x="73.09" y="77.49" size="1.778" layer="16" rot="MR90">5V</text>
-<text x="73.05" y="81.46" size="1.778" layer="16" rot="MR90">3.3V</text>
+<wire x1="1.35" y1="5.63" x2="80.72" y2="5.81" width="0" layer="20"/>
+<wire x1="80.72" y1="5.81" x2="80.45" y2="87.27" width="0" layer="20"/>
+<wire x1="80.45" y1="87.27" x2="1.37" y2="87.29" width="0" layer="20"/>
+<wire x1="1.37" y1="87.29" x2="1.35" y2="5.63" width="0" layer="20"/>
+<text x="74.45" y="70.25" size="1.778" layer="16" rot="MR0">_</text>
+<text x="75.07" y="77.55" size="1.778" layer="16" rot="MR0">5V</text>
+<text x="76.55" y="80.17" size="1.778" layer="16" rot="MR0">3.3V</text>
 <rectangle x1="65.84" y1="67.29" x2="70.79" y2="70.75" layer="16"/>
 <text x="9.13" y="53.21" size="1.778" layer="16" rot="MR0">+</text>
 <text x="42.26" y="19.85" size="1.016" layer="16" rot="MR0">GND</text>
 <text x="36.54" y="12.07" size="1.778" layer="16" rot="MR0">+</text>
+<text x="75.33" y="71.75" size="1.778" layer="16" rot="MR0">TX</text>
+<text x="75.49" y="74.74" size="1.778" layer="16" rot="MR0">RX</text>
 </plain>
 <attributes>

Commit message: BRD 8
Parts:
- L2-FCM1608-0603: device resistor:L3216C -> resistor:L4532M
Routing:
- net GND: track 557.1 -> 555.3 mm
